Commit message: Add lidar to sim

File: ros_ws/src/nanobot_description/urdf/robot.urdf.xacro (robot description, xacro)
@@ -3,4 +3,5 @@
   <xacro:arg name="sim_mode" default="false" />
   <xacro:include filename="robot_core.xacro" />
+  <xacro:include filename="lidar.xacro" />
   <xacro:if value="$(arg sim_mode)">
     <xacro:include filename="$(find nanobot_diffdrive)/description/gazebo_ros2_control.xacro" />

File: ros_ws/src/nanobot_description/urdf/robot_core.xacro (robot description, xacro)
@@ -5,5 +5,6 @@
   <xacro:property name="body_x_dim" value="0.14" />
   <xacro:property name="body_y_dim" value="0.14" />
-  <xacro:property name="body_z_dim" value="0.071" />
+  <xacro:property name="body_z_dim" value="0.058" /> <!-- check -->
+  <!-- <xacro:property name="body_z_dim" value="0.071" /> -->
   <!-- Wheel dimensions -->
   <xacro:property name="wheel_radius" value="0.03375" /> <!-- 67.5mm diameter -->
@@ -12,5 +13,5 @@
   <xacro:property name="caster_wheel_radius" value="${wheel_radius/2}" />
   <!-- Robot body and wheel mass -->
-  <xacro:property name="body_mass" value="0.906" />
+  <xacro:property name="body_mass" value="0.859" />
   <xacro:property name="wheel_mass" value="0.028" />
   <xacro:property name="caster_wheel_mass" value="0.008" />
@@ -29,9 +30,12 @@
   </xacro:macro>
   <!-- Materials -->
-  <material name="white">
-    <color rgba="1 1 1 1" />
+  <material name="yellow">
+    <color rgba="1 1 0 1" />
   </material>
   <material name="black">
     <color rgba="0 0 0 1" />
+  </material>
+  <material name="red">
+    <color rgba="1 0 0 1" />
   </material>
   <!-- Links and joints definition -->
@@ -50,5 +54,5 @@
         <box size="${body_x_dim} ${body_y_dim} ${body_z_dim}" />
       </geometry>
-      <material name="white" />
+      <material name="yellow" />
     </visual>
     <collision>
@@ -64,5 +68,5 @@
   </link>
   <gazebo reference="body_link">
-    <material>Gazebo/White</material>
+    <material>Gazebo/Yellow</material>
   </gazebo>
   <!-- Left wheel -->

Commit message: Add imu

File: ros_ws/src/nanobot_description/urdf/robot.urdf.xacro (robot description, xacro)
@@ -5,4 +5,5 @@
   <xacro:include filename="lidar.xacro" />
   <xacro:include filename="camera.xacro" />
+  <xacro:include filename="imu.xacro" />
   <xacro:if value="$(arg sim_mode)">
     <xacro:include filename="$(find nanobot_diffdrive)/description/gazebo_ros2_control.xacro" />

File: ros_ws/src/nanobot_description/urdf/robot_core.xacro (robot description, xacro)
@@ -5,11 +5,11 @@
   <xacro:property name="body_x_dim" value="0.14" />
   <xacro:property name="body_y_dim" value="0.14" />
-  <xacro:property name="body_z_dim" value="0.058" /> <!-- check -->
-  <!-- <xacro:property name="body_z_dim" value="0.071" /> -->
+  <xacro:property name="body_z_dim" value="0.076" />
+  <xacro:property name="body_z_offset" value="0.0175" />
   <!-- Wheel dimensions -->
   <xacro:property name="wheel_radius" value="0.03375" /> <!-- 67.5mm diameter -->
   <xacro:property name="wheel_length" value="0.025" />
   <xacro:property name="wheel_separation_from_body" value="0.0185" />
-  <xacro:property name="caster_wheel_radius" value="${wheel_radius/2}" />
+  <xacro:property name="caster_wheel_radius" value="${(wheel_radius - body_z_offset)/2}" />
   <!-- Robot body and wheel mass -->
   <xacro:property name="body_mass" value="0.859" />
@@ -46,5 +46,5 @@
     <parent link="base_link" />
     <child link="body_link" />
-    <origin xyz="-${body_x_dim/2} 0 0"/>
+    <origin xyz="-${body_x_dim/2} 0 -${body_z_offset}"/>
   </joint>
   <link name="body_link">
