Commit message: Improve robot sizes

File: ros_ws/src/nanobot_description/urdf/robot_core.xacro (robot description, xacro)
@@ -9,5 +9,5 @@
   <xacro:property name="wheel_radius" value="0.03375" /> <!-- 67.5mm diameter -->
   <xacro:property name="wheel_length" value="0.025" />
-  <xacro:property name="wheel_separation_from_body" value="0.0195" />
+  <xacro:property name="wheel_separation_from_body" value="0.0185" />
   <xacro:property name="caster_wheel_radius" value="${wheel_radius/2}" />
   <!-- Robot body and wheel mass -->

Commit message: Testing slam

File: ros_ws/src/nanobot_description/urdf/robot_core.xacro (robot description, xacro)
@@ -42,4 +42,12 @@
   <!-- Base link -->
   <link name="base_link"></link>
+  <!-- Base footprint -->
+ <joint name="base_footprint_joint" type="fixed">
+    <parent link="base_link"/>
+    <child link="base_footprint"/>
+    <origin xyz="0 0 0" rpy="0 0 0"/>
+  </joint>
+  <link name="base_footprint">
+  </link>
   <!-- Body -->
   <joint name="body_joint" type="fixed">

Commit message: Add room map

File: ros_ws/src/nanobot_description/urdf/robot_core.xacro (robot description, xacro)
@@ -43,5 +43,5 @@
   <link name="base_link"></link>
   <!-- Base footprint -->
- <joint name="base_footprint_joint" type="fixed">
+  <joint name="base_footprint_joint" type="fixed">
     <parent link="base_link"/>
     <child link="base_footprint"/>
