Commit message: Add depth camera

File: ros_ws/src/nanobot_description/urdf/camera.xacro (robot description, xacro)
@@ -2,15 +2,18 @@
 <robot xmlns:xacro="http://www.ros.org/wiki/xacro" name="nanobot">
   <!-- Camera specs -->
-  <xacro:property name="camera_x_dim" value="0.01" />
-  <xacro:property name="camera_y_dim" value="0.03" />
-  <xacro:property name="camera_z_dim" value="0.03" />
+  <xacro:property name="camera_x_dim" value="0.001" />
+  <xacro:property name="camera_y_dim" value="0.09" />
+  <xacro:property name="camera_z_dim" value="0.025" />
+  <xacro:property name="camera_height" value="0.06" />
+  <xacro:property name="center_offset" value="0.0175" />
   <!-- Links and joints definition -->
   <joint name="camera_joint" type="fixed">
     <parent link="body_link" />
     <child link="camera_link" />
-    <origin xyz="${body_x_dim + 0.02} 0 0.01" rpy="0 0 0" />
+    <origin xyz="${body_x_dim + camera_x_dim/2} ${center_offset} ${camera_height}" rpy="0 0 0" />
   </joint>
   <link name="camera_link">
     <visual>
+      <origin xyz="0 -${center_offset} 0" rpy="0 0 0" />
       <geometry>
         <box size="${camera_x_dim} ${camera_y_dim} ${camera_z_dim}" />

Commit message: Adapt description and diffdrive controller to new dimensions

File: ros_ws/src/nanobot_description/urdf/camera.xacro (robot description, xacro)
@@ -2,18 +2,19 @@
 <robot xmlns:xacro="http://www.ros.org/wiki/xacro" name="nanobot">
   <!-- Camera specs -->
-  <xacro:property name="camera_x_dim" value="0.001" />
+  <xacro:property name="camera_x_dim" value="0.025" />
   <xacro:property name="camera_y_dim" value="0.09" />
   <xacro:property name="camera_z_dim" value="0.025" />
-  <xacro:property name="camera_height" value="0.06" />
-  <xacro:property name="center_offset" value="0.0175" />
+  <xacro:property name="camera_x_offset" value="0.009" />
+  <xacro:property name="camera_height" value="0.085" />
+  <xacro:property name="sensor_offset" value="0.0175" />
   <!-- Links and joints definition -->
   <joint name="camera_joint" type="fixed">
     <parent link="body_link" />
     <child link="camera_link" />
-    <origin xyz="${body_x_dim + camera_x_dim/2} ${center_offset} ${camera_height}" rpy="0 0 0" />
+    <origin xyz="${body_x_dim + camera_x_offset} ${sensor_offset} ${camera_height}" rpy="0 0 0" />
   </joint>
   <link name="camera_link">
     <visual>
-      <origin xyz="0 -${center_offset} 0" rpy="0 0 0" />
+      <origin xyz="-${camera_x_dim/2} -${sensor_offset} 0" rpy="0 0 0" />
       <geometry>
         <box size="${camera_x_dim} ${camera_y_dim} ${camera_z_dim}" />

File: ros_ws/src/nanobot_description/urdf/robot.urdf.xacro (robot description, xacro)
@@ -3,7 +3,7 @@
   <xacro:arg name="sim_mode" default="false" />
   <xacro:include filename="robot_core.xacro" />
-  <xacro:include filename="lidar.xacro" />
+  <!-- <xacro:include filename="lidar.xacro" /> -->
   <xacro:include filename="camera.xacro" />
-  <xacro:include filename="imu.xacro" />
+  <!-- <xacro:include filename="imu.xacro" /> -->
   <xacro:if value="$(arg sim_mode)">
     <xacro:include filename="$(find nanobot_diffdrive)/description/gazebo_ros2_control.xacro" />

File: ros_ws/src/nanobot_description/urdf/robot_core.xacro (robot description, xacro)
@@ -3,17 +3,18 @@
   <xacro:include filename="inertial_macros.xacro" />
   <!-- Body dimensions -->
-  <xacro:property name="body_x_dim" value="0.14" />
-  <xacro:property name="body_y_dim" value="0.14" />
-  <xacro:property name="body_z_dim" value="0.076" />
-  <xacro:property name="body_z_offset" value="0.0175" />
+  <xacro:property name="body_x_dim" value="0.1425" />
+  <xacro:property name="body_y_dim" value="0.0765" />
+  <xacro:property name="body_z_dim" value="0.109" />
+  <xacro:property name="body_x_offset" value="0.02075" />
+  <xacro:property name="body_z_offset" value="0.01875" />
   <!-- Wheel dimensions -->
-  <xacro:property name="wheel_radius" value="0.03375" /> <!-- 67.5mm diameter -->
-  <xacro:property name="wheel_length" value="0.025" />
-  <xacro:property name="wheel_separation_from_body" value="0.0185" />
+  <xacro:property name="wheel_radius" value="0.033" /> <!-- 66mm diameter -->
+  <xacro:property name="wheel_length" value="0.018" />
+  <xacro:property name="wheel_separation_from_body" value="0.009" />
   <xacro:property name="caster_wheel_radius" value="${(wheel_radius - body_z_offset)/2}" />
   <!-- Robot body and wheel mass -->
-  <xacro:property name="body_mass" value="0.859" />
+  <xacro:property name="body_mass" value="0.941" />
   <xacro:property name="wheel_mass" value="0.028" />
-  <xacro:property name="caster_wheel_mass" value="0.008" />
+  <xacro:property name="caster_wheel_mass" value="0.041" />
   <!-- Moments of intertia of the wheel -->
   <xacro:macro name="inertia_wheel">
@@ -54,5 +55,5 @@
     <parent link="base_link" />
     <child link="body_link" />
-    <origin xyz="-${body_x_dim/2} 0 -${body_z_offset}"/>
+    <origin xyz="-${body_x_offset} 0 -${body_z_offset}"/>
   </joint>
   <link name="body_link">
@@ -138,13 +139,13 @@
     <mu2 value="0.2" /> -->
   </gazebo>
-  <!-- Back caster wheel -->
-  <joint name="back_caster_wheel_joint" type="fixed">
+  <!-- Caster wheel -->
+  <joint name="caster_wheel_joint" type="fixed">
       <parent link="body_link"/>
-      <child link="back_caster_wheel_link"/>
+      <child link="caster_wheel_link"/>
       <origin
-        xyz="${caster_wheel_radius} 0 -${caster_wheel_radius}"
+        xyz="${body_x_dim - caster_wheel_radius} 0 -${caster_wheel_radius}"
         rpy="0 0 0"/>
   </joint>
-  <link name="back_caster_wheel_link">
+  <link name="caster_wheel_link">
     <visual>
       <geometry>
@@ -160,32 +161,5 @@
     <xacro:inertia_caster_wheel />
   </link>
-  <gazebo reference="back_caster_wheel_link">
-    <material>Gazebo/Black</material>
-    <mu1 value="0.001"/>
-    <mu2 value="0.001"/>
-  </gazebo>
-  <!-- Front caster wheel -->
-  <joint name="front_caster_wheel_joint" type="fixed">
-      <parent link="body_link"/>
-      <child link="front_caster_wheel_link"/>
-      <origin
-        xyz="${body_x_dim - caster_wheel_radius} 0 -${caster_wheel_radius}"
-        rpy="0 0 0"/>
-  </joint>
-  <link name="front_caster_wheel_link">
-    <visual>
-      <geometry>
-        <sphere radius="${caster_wheel_radius}" />
-      </geometry>
-      <material name="black"/>
-    </visual>
-    <collision>
-      <geometry>
-        <sphere radius="${caster_wheel_radius}" />
-      </geometry>
-    </collision>
-    <xacro:inertia_caster_wheel />
-  </link>
-  <gazebo reference="front_caster_wheel_link">
+  <gazebo reference="caster_wheel_link">
     <material>Gazebo/Black</material>
     <mu1 value="0.001"/>

File: ros_ws/src/nanobot_diffdrive/description/ros2_control.xacro (robot description, xacro)
@@ -6,7 +6,7 @@
       <param name="left_wheel_name">left_wheel_joint</param>
       <param name="right_wheel_name">right_wheel_joint</param>
-      <param name="left_motor_id">1</param>
-      <param name="right_motor_id">2</param>
-      <param name="velocity_limit">250</param>
+      <param name="left_motor_id">2</param>
+      <param name="right_motor_id">1</param>
+      <param name="velocity_limit">1023</param>
       <param name="rpm_per_unit">0.229</param> <!-- see https://emanual.robotis.com/docs/en/dxl/x/xl430-w250/#goal-velocity -->
       <param name="deg_per_pulse">0.088</param> <!-- see https://emanual.robotis.com/docs/en/dxl/x/xl430-w250/#goal-position -->
