Commit message: Fix imu issues, enable ekf

File: ros/nanobot_description/urdf/imu.xacro (robot description, xacro)
@@ -5,9 +5,9 @@
   <xacro:property name="imu_body_z_offset" value="0.004" />
   <!-- Links and joints definition -->
-  <joint name="imu_base_joint" type="fixed">
+  <joint name="imu_joint" type="fixed">
     <parent link="base_link" />
-    <child link="imu_base_link" />
+    <child link="imu_link" />
     <origin xyz="0 0 ${body_z_dim - body_z_offset - imu_body_z_offset - imu_z_dim}" rpy="0 0 ${pi/2}" />
   </joint>
-  <link name="imu_base_link" />
+  <link name="imu_link" />
 </robot>

File: ros/nanobot_description/urdf/robot.urdf.xacro (robot description, xacro)
@@ -5,5 +5,5 @@
   <!-- <xacro:include filename="lidar.xacro" /> -->
   <xacro:include filename="camera.xacro" />
-  <!-- <xacro:include filename="imu.xacro" /> -->
+  <xacro:include filename="imu.xacro" />
   <xacro:if value="$(arg sim_mode)">
     <xacro:include filename="$(find nanobot_diffdrive)/description/gazebo_ros2_control.xacro" />
