Commit message: Add diffdrive support for multiple wheels

File: ros/nanobot_description/urdf/robot_core.xacro (robot description, xacro)
@@ -79,8 +79,12 @@
     <material>Gazebo/Yellow</material>
   </gazebo>
-  <!-- Left wheel -->
-  <joint name="left_wheel_joint" type="continuous">
+  <!-- Front left wheel -->
+  <!-- TODO: Enable front wheels -->
+  <!-- Front right wheel -->
+  <!-- TODO: Enable front wheels -->
+  <!-- Rear left wheel -->
+  <joint name="rear_left_wheel_joint" type="continuous">
     <parent link="base_link" />
-    <child link="left_wheel_link" />
+    <child link="rear_left_wheel_link" />
     <origin
       xyz="0 ${body_y_dim/2 + wheel_length/2 + wheel_separation_from_body} 0"
@@ -90,5 +94,5 @@
     <!-- <dynamics damping="1.0" friction="1.0" /> -->
   </joint>
-  <link name="left_wheel_link">
+  <link name="rear_left_wheel_link">
     <visual>
       <geometry>
@@ -104,13 +108,13 @@
     <xacro:inertia_wheel />
   </link>
-  <gazebo reference="left_wheel_link">
+  <gazebo reference="rear_left_wheel_link">
     <material>Gazebo/Black</material>
     <!-- <mu1 value="0.2" />
     <mu2 value="0.2" /> -->
   </gazebo>
-  <!-- Right wheel -->
-  <joint name="right_wheel_joint" type="continuous">
+  <!-- Rear right wheel -->
+  <joint name="rear_right_wheel_joint" type="continuous">
     <parent link="base_link" />
-    <child link="right_wheel_link" />
+    <child link="rear_right_wheel_link" />
     <origin
       xyz="0 -${body_y_dim/2 + wheel_length/2 + wheel_separation_from_body} 0"
@@ -120,5 +124,5 @@
     <!-- <dynamics damping="1.0" friction="1.0" /> -->
   </joint>
-  <link name="right_wheel_link">
+  <link name="rear_right_wheel_link">
     <visual>
       <geometry>
@@ -134,5 +138,5 @@
     <xacro:inertia_wheel />
   </link>
-  <gazebo reference="right_wheel_link">
+  <gazebo reference="rear_right_wheel_link">
     <material>Gazebo/Black</material>
     <!-- <mu1 value="0.2" />
@@ -140,4 +144,5 @@
   </gazebo>
   <!-- Caster wheel -->
+  <!-- TODO: Enable front wheels -->
   <joint name="caster_wheel_joint" type="fixed">
       <parent link="body_link"/>

File: ros/nanobot_diffdrive/description/gazebo_ros2_control.xacro (robot description, xacro)
@@ -5,5 +5,6 @@
       <plugin>ign_ros2_control/IgnitionSystem</plugin>
     </hardware>
-    <joint name="left_wheel_joint">
+    <!-- TODO: Enable front wheels -->
+    <!-- <joint name="front_left_wheel_joint">
       <command_interface name="velocity">
         <param name="min">-10</param>
@@ -13,5 +14,21 @@
       <state_interface name="position" />
     </joint>
-    <joint name="right_wheel_joint">
+    <joint name="front_right_wheel_joint">
+      <command_interface name="velocity">
+        <param name="min">-10</param>
+        <param name="max">10</param>
+      </command_interface>
+      <state_interface name="velocity" />
+      <state_interface name="position" />
+    </joint> -->
+    <joint name="rear_left_wheel_joint">
+      <command_interface name="velocity">
+        <param name="min">-10</param>
+        <param name="max">10</param>
+      </command_interface>
+      <state_interface name="velocity" />
+      <state_interface name="position" />
+    </joint>
+    <joint name="rear_right_wheel_joint">
       <command_interface name="velocity">
         <param name="min">-10</param>

File: ros/nanobot_diffdrive/description/ros2_control.xacro (robot description, xacro)
@@ -4,8 +4,17 @@
     <hardware>
       <plugin>nanobot_diffdrive/NanobotDiffDriveHardware</plugin>
-      <param name="left_wheel_name">left_wheel_joint</param>
-      <param name="right_wheel_name">right_wheel_joint</param>
-      <param name="left_motor_id">2</param>
-      <param name="right_motor_id">1</param>
+      <param name="left_wheel_names">rear_left_wheel_joint</param>
+      <param name="right_wheel_names">rear_right_wheel_joint</param>
+      <param name="left_motor_ids">2</param>
+      <param name="right_motor_ids">1</param>
+      <param name="left_wheel_signs">1</param>
+      <param name="right_wheel_signs">-1</param>
+      <!-- TODO: Enable front wheels -->
+      <!-- <param name="left_wheel_names">front_left_wheel_joint,rear_left_wheel_joint</param>
+      <param name="right_wheel_names">front_right_wheel_joint,rear_right_wheel_joint</param>
+      <param name="left_motor_ids">4,2</param>
+      <param name="right_motor_ids">3,1</param>
+      <param name="left_wheel_signs">-1,1</param>
+      <param name="right_wheel_signs">1,-1</param> -->
       <param name="velocity_limit">1023</param>
       <param name="rpm_per_unit">0.229</param> <!-- see https://emanual.robotis.com/docs/en/dxl/x/xl430-w250/#goal-velocity -->
@@ -15,10 +24,21 @@
       <param name="baud_rate">57600</param>
     </hardware>
-    <joint name="left_wheel_joint">
+    <!-- TODO: Enable front wheels -->
+    <!-- <joint name="front_left_wheel_joint">
       <command_interface name="velocity" />
       <state_interface name="position" />
       <state_interface name="velocity" />
     </joint>
-    <joint name="right_wheel_joint">
+    <joint name="front_right_wheel_joint">
+      <command_interface name="velocity" />
+      <state_interface name="position" />
+      <state_interface name="velocity" />
+    </joint> -->
+    <joint name="rear_left_wheel_joint">
+      <command_interface name="velocity" />
+      <state_interface name="position" />
+      <state_interface name="velocity" />
+    </joint>
+    <joint name="rear_right_wheel_joint">
       <command_interface name="velocity" />
       <state_interface name="position" />
