Commit message: Update sizes and enable front wheels

File: ros/nanobot_description/urdf/camera.xacro (robot description, xacro)
@@ -5,6 +5,6 @@
   <xacro:property name="camera_y_dim" value="0.09" />
   <xacro:property name="camera_z_dim" value="0.025" />
-  <xacro:property name="camera_x_offset" value="0.009" />
-  <xacro:property name="camera_height" value="0.085" />
+  <xacro:property name="camera_x_offset" value="0.001" />
+  <xacro:property name="camera_height" value="0.0875" />
   <xacro:property name="sensor_offset" value="0.0175" />
   <!-- Links and joints definition -->
@@ -12,5 +12,5 @@
     <parent link="body_link" />
     <child link="camera_link" />
-    <origin xyz="${body_x_dim + camera_x_offset} ${sensor_offset} ${camera_height}" rpy="0 0 0" />
+    <origin xyz="${body_x_dim/2 + camera_x_offset} ${sensor_offset} ${camera_height}" rpy="0 0 0" />
   </joint>
   <link name="camera_link">

File: ros/nanobot_description/urdf/imu.xacro (robot description, xacro)
@@ -2,11 +2,11 @@
 <robot xmlns:xacro="http://www.ros.org/wiki/xacro" name="nanobot">
   <!-- IMU specs -->
-  <xacro:property name="imu_z_dim" value="0.002" />
-  <xacro:property name="imu_body_z_offset" value="0.004" />
+  <xacro:property name="imu_x_offset" value="0.004" />
+  <xacro:property name="imu_height" value="0.06125" />
   <!-- Links and joints definition -->
   <joint name="imu_joint" type="fixed">
-    <parent link="base_link" />
+    <parent link="body_link" />
     <child link="imu_link" />
-    <origin xyz="0 0 ${body_z_dim - body_z_offset - imu_body_z_offset - imu_z_dim}" rpy="0 0 ${pi/2}" />
+    <origin xyz="${body_x_dim/2 - imu_x_offset} 0 ${imu_height}" rpy="0 0 ${pi/2}" />
   </joint>
   <link name="imu_link" />

File: ros/nanobot_description/urdf/robot_core.xacro (robot description, xacro)
@@ -3,18 +3,16 @@
   <xacro:include filename="inertial_macros.xacro" />
   <!-- Body dimensions -->
-  <xacro:property name="body_x_dim" value="0.1425" />
+  <xacro:property name="body_x_dim" value="0.152" />
   <xacro:property name="body_y_dim" value="0.0765" />
-  <xacro:property name="body_z_dim" value="0.109" />
-  <xacro:property name="body_x_offset" value="0.02075" />
-  <xacro:property name="body_z_offset" value="0.01875" />
+  <xacro:property name="body_z_dim" value="0.110" />
+  <xacro:property name="body_z_offset" value="0.01425" />
   <!-- Wheel dimensions -->
   <xacro:property name="wheel_radius" value="0.033" /> <!-- 66mm diameter -->
   <xacro:property name="wheel_length" value="0.018" />
-  <xacro:property name="wheel_separation_from_body" value="0.009" />
-  <xacro:property name="caster_wheel_radius" value="${(wheel_radius - body_z_offset)/2}" />
+  <xacro:property name="wheel_x_offset" value="0.05875" />
+  <xacro:property name="wheel_y_offset" value="0.00825" />
   <!-- Robot body and wheel mass -->
-  <xacro:property name="body_mass" value="0.941" />
+  <xacro:property name="body_mass" value="1.256" />
   <xacro:property name="wheel_mass" value="0.028" />
-  <xacro:property name="caster_wheel_mass" value="0.041" />
   <!-- Moments of intertia of the wheel -->
   <xacro:macro name="inertia_wheel">
@@ -23,10 +21,4 @@
       <origin xyz="0 0 0" rpy="0 0 0" />
     </xacro:inertial_cylinder>
-  </xacro:macro>
-  <!-- Moments of intertia of the caster wheel -->
-  <xacro:macro name="inertia_caster_wheel">
-    <xacro:inertial_sphere mass="${caster_wheel_mass}" radius="${caster_wheel_radius}">
-      <origin xyz="0 0 0" rpy="0 0 0" />
-    </xacro:inertial_sphere>
   </xacro:macro>
   <!-- Materials -->
@@ -41,23 +33,23 @@
   </material>
   <!-- Links and joints definition -->
+  <!-- TODO: Enable base footprint  -->
+  <!-- Base footprint -->
+  <!-- <joint name="base_joint" type="fixed">
+    <parent link="base_footprint"/>
+    <child link="base_link"/>
+    <origin xyz="0 0 ${wheel_radius}" rpy="0 0 0"/>
+  </joint>
+  <link name="base_footprint"></link> -->
   <!-- Base link -->
   <link name="base_link"></link>
-  <!-- Base footprint -->
-  <joint name="base_footprint_joint" type="fixed">
-    <parent link="base_link"/>
-    <child link="base_footprint"/>
-    <origin xyz="0 0 0" rpy="0 0 0"/>
-  </joint>
-  <link name="base_footprint">
-  </link>
   <!-- Body -->
   <joint name="body_joint" type="fixed">
     <parent link="base_link" />
     <child link="body_link" />
-    <origin xyz="-${body_x_offset} 0 -${body_z_offset}"/>
+    <origin xyz="0 0 -${body_z_offset}"/>
   </joint>
   <link name="body_link">
     <visual>
-      <origin xyz="${body_x_dim/2} 0 ${body_z_dim/2}" rpy="0 0 0" />
+      <origin xyz="0 0 ${body_z_dim/2}" rpy="0 0 0" />
       <geometry>
         <box size="${body_x_dim} ${body_y_dim} ${body_z_dim}" />
@@ -66,5 +58,5 @@
     </visual>
     <collision>
-      <origin xyz="${body_x_dim/2} 0 ${body_z_dim/2}" rpy="0 0 0" />
+      <origin xyz="0 0 ${body_z_dim/2}" rpy="0 0 0" />
       <geometry>
         <box size="${body_x_dim} ${body_y_dim} ${body_z_dim}" />
@@ -73,5 +65,5 @@
     <xacro:inertial_box mass="${body_mass}" x="${body_x_dim}" y="${body_y_dim}"
       z="${body_z_dim}">
-      <origin xyz="${body_x_dim/2} 0 ${body_z_dim/2}" rpy="0 0 0" />
+      <origin xyz="0 0 ${body_z_dim/2}" rpy="0 0 0" />
     </xacro:inertial_box>
   </link>
@@ -80,7 +72,63 @@
   </gazebo>
   <!-- Front left wheel -->
-  <!-- TODO: Enable front wheels -->
+  <joint name="front_left_wheel_joint" type="continuous">
+    <parent link="base_link" />
+    <child link="front_left_wheel_link" />
+    <origin
+      xyz="${wheel_x_offset} ${body_y_dim/2 + wheel_length/2 + wheel_y_offset} 0"
+      rpy="-${pi/2} 0 0" />
+    <axis xyz="0 0 1" />
+    <limit effort="100" velocity="100" />
+    <!-- <dynamics damping="1.0" friction="1.0" /> -->
+  </joint>
+  <link name="front_left_wheel_link">
+    <visual>
+      <geometry>
+        <cylinder length="${wheel_length}" radius="${wheel_radius}" />
+      </geometry>
+      <material name="black" />
+    </visual>
+    <collision>
+      <geometry>
+        <sphere radius="${wheel_radius}" />
+      </geometry>
+    </collision>
+    <xacro:inertia_wheel />
+  </link>
+  <gazebo reference="front_left_wheel_link">
+    <material>Gazebo/Black</material>
+    <!-- <mu1 value="0.2" />
+    <mu2 value="0.2" /> -->
+  </gazebo>
   <!-- Front right wheel -->
-  <!-- TODO: Enable front wheels -->
+  <joint name="front_right_wheel_joint" type="continuous">
+    <parent link="base_link" />
+    <child link="front_right_wheel_link" />
+    <origin
+      xyz="${wheel_x_offset} -${body_y_dim/2 + wheel_length/2 + wheel_y_offset} 0"
+      rpy="${pi/2} 0 0" />
+    <axis xyz="0 0 -1" />
+    <limit effort="100" velocity="100" />
+    <!-- <dynamics damping="1.0" friction="1.0" /> -->
+  </joint>
+  <link name="front_right_wheel_link">
+    <visual>
+      <geometry>
+        <cylinder length="${wheel_length}" radius="${wheel_radius}" />
+      </geometry>
+      <material name="black" />
+    </visual>
+    <collision>
+      <geometry>
+        <sphere radius="${wheel_radius}" />
+      </geometry>
+    </collision>
+    <xacro:inertia_wheel />
+  </link>
+  <gazebo reference="front_right_wheel_link">
+    <material>Gazebo/Black</material>
+    <!-- <mu1 value="0.2" />
+    <mu2 value="0.2" /> -->
+  </gazebo>
   <!-- Rear left wheel -->
   <joint name="rear_left_wheel_joint" type="continuous">
@@ -88,5 +136,5 @@
     <child link="rear_left_wheel_link" />
     <origin
-      xyz="0 ${body_y_dim/2 + wheel_length/2 + wheel_separation_from_body} 0"
+      xyz="-${wheel_x_offset} ${body_y_dim/2 + wheel_length/2 + wheel_y_offset} 0"
       rpy="-${pi/2} 0 0" />
     <axis xyz="0 0 1" />
@@ -118,5 +166,5 @@
     <child link="rear_right_wheel_link" />
     <origin
-      xyz="0 -${body_y_dim/2 + wheel_length/2 + wheel_separation_from_body} 0"
+      xyz="-${wheel_x_offset} -${body_y_dim/2 + wheel_length/2 + wheel_y_offset} 0"
       rpy="${pi/2} 0 0" />
     <axis xyz="0 0 -1" />
@@ -143,31 +191,3 @@
     <mu2 value="0.2" /> -->
   </gazebo>
-  <!-- Caster wheel -->
-  <!-- TODO: Enable front wheels -->
-  <joint name="caster_wheel_joint" type="fixed">
-      <parent link="body_link"/>
-      <child link="caster_wheel_link"/>
-      <origin
-        xyz="${body_x_dim - caster_wheel_radius} 0 -${caster_wheel_radius}"
-        rpy="0 0 0"/>
-  </joint>
-  <link name="caster_wheel_link">
-    <visual>
-      <geometry>
-        <sphere radius="${caster_wheel_radius}" />
-      </geometry>
-      <material name="black"/>
-    </visual>
-    <collision>
-      <geometry>
-        <sphere radius="${caster_wheel_radius}" />
-      </geometry>
-    </collision>
-    <xacro:inertia_caster_wheel />
-  </link>
-  <gazebo reference="caster_wheel_link">
-    <material>Gazebo/Black</material>
-    <mu1 value="0.001"/>
-    <mu2 value="0.001"/>
-  </gazebo>
 </robot>

File: ros/nanobot_diffdrive/description/gazebo_ros2_control.xacro (robot description, xacro)
@@ -5,6 +5,5 @@
       <plugin>ign_ros2_control/IgnitionSystem</plugin>
     </hardware>
-    <!-- TODO: Enable front wheels -->
-    <!-- <joint name="front_left_wheel_joint">
+    <joint name="front_left_wheel_joint">
       <command_interface name="velocity">
         <param name="min">-10</param>
@@ -21,5 +20,5 @@
       <state_interface name="velocity" />
       <state_interface name="position" />
-    </joint> -->
+    </joint>
     <joint name="rear_left_wheel_joint">
       <command_interface name="velocity">

File: ros/nanobot_diffdrive/description/ros2_control.xacro (robot description, xacro)
@@ -4,17 +4,10 @@
     <hardware>
       <plugin>nanobot_diffdrive/NanobotDiffDriveHardware</plugin>
-      <param name="left_wheel_names">rear_left_wheel_joint</param>
-      <param name="right_wheel_names">rear_right_wheel_joint</param>
-      <param name="left_motor_ids">2</param>
-      <param name="right_motor_ids">1</param>
-      <param name="left_wheel_signs">1</param>
-      <param name="right_wheel_signs">-1</param>
-      <!-- TODO: Enable front wheels -->
-      <!-- <param name="left_wheel_names">front_left_wheel_joint,rear_left_wheel_joint</param>
+      <param name="left_wheel_names">front_left_wheel_joint,rear_left_wheel_joint</param>
       <param name="right_wheel_names">front_right_wheel_joint,rear_right_wheel_joint</param>
-      <param name="left_motor_ids">4,2</param>
-      <param name="right_motor_ids">3,1</param>
-      <param name="left_wheel_signs">-1,1</param>
-      <param name="right_wheel_signs">1,-1</param> -->
+      <param name="left_motor_ids">1,3</param>
+      <param name="right_motor_ids">2,4</param>
+      <param name="left_wheel_signs">1,1</param>
+      <param name="right_wheel_signs">-1,-1</param>
       <param name="velocity_limit">1023</param>
       <param name="rpm_per_unit">0.229</param> <!-- see https://emanual.robotis.com/docs/en/dxl/x/xl430-w250/#goal-velocity -->
@@ -24,6 +17,5 @@
       <param name="baud_rate">57600</param>
     </hardware>
-    <!-- TODO: Enable front wheels -->
-    <!-- <joint name="front_left_wheel_joint">
+    <joint name="front_left_wheel_joint">
       <command_interface name="velocity" />
       <state_interface name="position" />
@@ -34,5 +26,5 @@
       <state_interface name="position" />
       <state_interface name="velocity" />
-    </joint> -->
+    </joint>
     <joint name="rear_left_wheel_joint">
       <command_interface name="velocity" />
