Commit message: Add suport to rplidar c1

File: ros/nanobot_description/urdf/lidar.xacro (robot description, xacro)
@@ -2,65 +2,67 @@
 <robot xmlns:xacro="http://www.ros.org/wiki/xacro" name="nanobot">
   <!-- LIDAR specs -->
-  <xacro:property name="ldlidar_base_x_dim" value="0.039" />
-  <xacro:property name="ldlidar_base_y_dim" value="0.039" />
-  <xacro:property name="ldlidar_base_z_dim" value="0.0222" />
-  <xacro:property name="ldlidar_link_height" value="0.0126" />
-  <xacro:property name="ldlidar_link_radius" value="0.017645" />
-  <xacro:property name="ldlidar_mass" value="0.047" />
+  <xacro:property name="lidar_base_x_dim" value="0.0556" />
+  <xacro:property name="lidar_base_y_dim" value="0.0556" />
+  <xacro:property name="lidar_base_z_dim" value="0.0231" />
+  <xacro:property name="lidar_x_offset" value="0.0355" />
+  <xacro:property name="lidar_link_height" value="0.0182" />
+  <xacro:property name="lidar_link_radius" value="0.0255" />
+  <xacro:property name="lidar_laser_height" value="0.0067" />
+  <xacro:property name="lidar_mass" value="0.11" />
   <!-- Links and joints definition -->
   <!-- Base -->
-  <joint name="ldlidar_base_joint" type="fixed">
+  <joint name="lidar_base_joint" type="fixed">
     <parent link="body_link" />
-    <child link="ldlidar_base_link" />
-    <origin xyz="${body_x_dim/2} 0 ${body_z_dim}" rpy="0 0 ${pi/2}" />
+    <child link="lidar_base_link" />
+    <origin xyz="${-body_x_dim/2 + lidar_x_offset} 0 ${body_z_dim}" rpy="0 0 ${-pi/2}" />
   </joint>
-  <link name="ldlidar_base_link">
+  <link name="lidar_base_link">
     <visual>
-      <origin xyz="0 0 ${ldlidar_base_z_dim/2}" rpy="0 0 0" />
+      <origin xyz="0 0 ${lidar_base_z_dim/2}" rpy="0 0 0" />
       <geometry>
-        <box size="${ldlidar_base_x_dim} ${ldlidar_base_y_dim} ${ldlidar_base_z_dim}" />
+        <box size="${lidar_base_x_dim} ${lidar_base_y_dim} ${lidar_base_z_dim}" />
       </geometry>
       <material name="red" />
     </visual>
     <collision>
-      <origin xyz="0 0 ${ldlidar_base_z_dim/2}" rpy="0 0 0" />
+      <origin xyz="0 0 ${lidar_base_z_dim/2}" rpy="0 0 0" />
       <geometry>
-        <box size="${ldlidar_base_x_dim} ${ldlidar_base_y_dim} ${ldlidar_base_z_dim}" />
+        <box size="${lidar_base_x_dim} ${lidar_base_y_dim} ${lidar_base_z_dim}" />
       </geometry>
     </collision>
-    <xacro:inertial_box mass="${ldlidar_mass/2}" x="${ldlidar_base_x_dim}" y="${ldlidar_base_y_dim}"
-      z="${ldlidar_base_z_dim}">
-      <origin xyz="0 0 ${ldlidar_base_z_dim/2}" rpy="0 0 0" />
+    <xacro:inertial_box mass="${lidar_mass/2}" x="${lidar_base_x_dim}" y="${lidar_base_y_dim}"
+      z="${lidar_base_z_dim}">
+      <origin xyz="0 0 ${lidar_base_z_dim/2}" rpy="0 0 0" />
     </xacro:inertial_box>
   </link>
   <!-- Link -->
-  <joint name="ldlidar_link_joint" type="fixed">
-    <parent link="ldlidar_base_link" />
-    <child link="ldlidar_link" />
-    <origin xyz="0 0 ${ldlidar_base_z_dim + ldlidar_link_height/2}" rpy="0 0 0" />
+  <joint name="lidar_link_joint" type="fixed">
+    <parent link="lidar_base_link" />
+    <child link="lidar_link" />
+    <origin xyz="0 0 ${lidar_base_z_dim + lidar_laser_height}" rpy="0 0 0" />
   </joint>
-  <link name="ldlidar_link">
+  <link name="lidar_link">
     <visual>
-      <origin xyz="0 0 0" rpy="0 0 0" />
+      <origin xyz="0 0 ${lidar_link_height/2 - lidar_laser_height}" rpy="0 0 0" />
       <geometry>
-        <cylinder length="${ldlidar_link_height}" radius="${ldlidar_link_radius}" />
+        <cylinder length="${lidar_link_height}" radius="${lidar_link_radius}" />
       </geometry>
       <material name="red" />
     </visual>
     <collision>
-      <origin xyz="0 0 0" rpy="0 0 0" />
+      <origin xyz="0 0 ${lidar_link_height/2 - lidar_laser_height}" rpy="0 0 0" />
       <geometry>
-        <cylinder length="${ldlidar_link_height}" radius="${ldlidar_link_radius}" />
+        <cylinder length="${lidar_link_height}" radius="${lidar_link_radius}" />
       </geometry>
     </collision>
-    <xacro:inertial_cylinder mass="${ldlidar_mass/2}" length="${ldlidar_link_height}" radius="${ldlidar_link_radius}">
-      <origin xyz="0 0 0" rpy="0 0 0" />
+    <xacro:inertial_cylinder mass="${lidar_mass/2}" length="${lidar_link_height}" radius="${lidar_link_radius}">
+      <origin xyz="0 0 ${lidar_link_height/2 - lidar_laser_height}" rpy="0 0 0" />
     </xacro:inertial_cylinder>
   </link>
   <!-- Gazebo -->
-  <gazebo reference="ldlidar_base_link">
+  <gazebo reference="lidar_base_link">
     <material>Gazebo/Red</material>
   </gazebo>
-  <gazebo reference="ldlidar_link">
+  <gazebo reference="lidar_link">
     <material>Gazebo/Red</material>
     <sensor name="laser" type="gpu_lidar">
@@ -77,10 +79,10 @@
         </scan>
         <range>
-          <min>0.02</min>
+          <min>0.05</min>
           <max>12</max>
         </range>
       </lidar>
       <topic>lidar/scan</topic>
-      <gz_frame_id>ldlidar_link</gz_frame_id>
+      <gz_frame_id>lidar_link</gz_frame_id>
     </sensor>
   </gazebo>

File: ros/nanobot_description/urdf/robot.urdf.xacro (robot description, xacro)
@@ -3,5 +3,5 @@
   <xacro:arg name="sim_mode" default="false" />
   <xacro:include filename="robot_core.xacro" />
-  <!-- <xacro:include filename="lidar.xacro" /> -->
+  <xacro:include filename="lidar.xacro" />
   <xacro:include filename="camera.xacro" />
   <xacro:include filename="imu.xacro" />

File: ros/nanobot_description/urdf/robot_core.xacro (robot description, xacro)
@@ -13,5 +13,5 @@
   <xacro:property name="wheel_y_offset" value="0.00825" />
   <!-- Robot body and wheel mass -->
-  <xacro:property name="body_mass" value="1.256" />
+  <xacro:property name="body_mass" value="1.146" />
   <xacro:property name="wheel_mass" value="0.028" />
   <!-- Moments of intertia of the wheel -->
